File: Horticulture-rev3.0.1.0/Horticulture.kicad_pcb (KiCad board)
At the start: 2 copper layers, 220 x 22 mm, 51 parts, among them J2 Conn_02x05_Odd_Even, J3 Conn_01x04_Male, J4 Conn_01x04_Male, SW1 SW-I2C, SW2 Rotary_Encoder_Switch, U1 TLE4309, U2 TLE4309, U3 TLE4309, U4 TLE4309, U5 AMS1117-3.3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

Commit message: Working on sensor board
Other:
- board text added: "Horticulture rev 3.0.1.0"
Changed lines of the file:
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@@
   (general
     (thickness 1.6)
-    (drawings 8)
+    (drawings 9)
     (tracks 776)
     (zones 0)
@@
   (layers
     (0 F.Cu signal)
-    (31 B.Cu signal)
-    (32 B.Adhes user)
+    (31 B.Cu signal hide)
+    (32 B.Adhes user hide)
     (33 F.Adhes user)
     (34 B.Paste user)
@@
     (36 B.SilkS user)
     (37 F.SilkS user)
-    (38 B.Mask user)
+    (38 B.Mask user hide)
     (39 F.Mask user)
     (40 Dwgs.User user)
@@
       (outputformat 1)
       (mirror false)
-      (drillshape 1)
+      (drillshape 0)
       (scaleselection 1)
-      (outputdirectory ""))
+      (outputdirectory "plots/"))
   )
   (net 0 "")
@@
     )
   )
+  (gr_text "Horticulture\nrev 3.0.1.0" (at 94.025 95.825 180) (layer B.SilkS)
+    (effects (font (size 1.5 1.5) (thickness 0.15)) (justify mirror))
+  )
   (gr_circle (center 258.5 100.5) (end 259.51 100.5) (layer Edge.Cuts) (width 0.1))
