File: Horticulture-sensor-rev1.0/HorticultureSensor.kicad_pcb (KiCad board)
At the start: 2 copper layers, 46.9 x 34.8 mm, 24 parts, among them J1 Conn_01x04, J2 Conn_02x05_Odd_Even, J3 Conn_01x03, J4 Conn_01x04, J5 Conn_01x03, J6 Conn_01x02, J7 Conn_01x02, J8 Conn_01x02, Q1 IRLML2030TRPBF, Q2 IRLML2030TRPBF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

Commit message: Somethings updated
Parts:
- moved R1 1.93 mm to (181.3, 120.1), turned to 180 degrees
Connections:
- J2 pad 6: Net-(J2-Pad6) -> (no net)
- J2 pad 7: Net-(J2-Pad7) -> (no net)
- J2 pad 8: Net-(J2-Pad8) -> (no net)
- J2 pad 9: Net-(J2-Pad9) -> (no net)
- Q1 pad 1: Net-(Q1-Pad1) -> mosfet0
- Q2 pad 1: Net-(Q2-Pad1) -> mosfet1
- R1 pad 1: Net-(Q1-Pad1) -> mosfet0
- R1 pad 2: mosfet0 -> 12V-
- R2 pad 1: Net-(Q2-Pad1) -> mosfet1
- R2 pad 2: mosfet1 -> 12V-
- U1 pad 1: Net-(U1-Pad1) -> (no net)
- U1 pad 14: Net-(U1-Pad14) -> (no net)
- U1 pad 2: Net-(U1-Pad2) -> (no net)
- U1 pad 3: Net-(U1-Pad3) -> (no net)
Routing:
- net mosfet1: track 34.0 -> 40.6 mm
- net 12V-: track 78.9 -> 84.8 mm
- net mosfet0: track 23.8 -> 29.0 mm
- net Net-(Q2-Pad1): track 2.80 -> 0.00 mm
- net Net-(Q1-Pad1): track 2.30 -> 0.00 mm
Other:
- board text added: "Horticulture Sensor rev 1.0.1"
- board text removed: "Horticulture Sensor rev 1.0"
