File: Horticulture.kicad_pcb (KiCad board)
At the start: 2 copper layers, 220 x 22 mm, 59 parts, among them J2 Conn_02x05_Odd_Even, J3 Conn_01x04_Male, J4 Conn_01x04_Male, SW1 SW-I2C, SW2 Rotary_Encoder_Switch, U1 TLE4309, U2 TLE4309, U3 TLE4309, U4 TLE4309, U6 STM32F030F4Px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

Commit message: Added footprint to new resistors
Parts:
- added R11: 10K2, Resistor_SMD:R_0603_1608Metric, B.Cu at (69.8, 83.8)
- added R12: 10K2, Resistor_SMD:R_0603_1608Metric, F.Cu at (190.5, 67.3)
- added R13: 10K2, Resistor_SMD:R_0603_1608Metric, F.Cu at (194.5, 64.8)
- added R14: 10K2, Resistor_SMD:R_0603_1608Metric, F.Cu at (190.5, 69.8)
- added R15: 10K2, Resistor_SMD:R_0603_1608Metric, F.Cu at (194.5, 67.3)
- added R16: 10K2, Resistor_SMD:R_0603_1608Metric, F.Cu at (198.5, 64.8)
- added R17: 10K2, Resistor_SMD:R_0603_1608Metric, F.Cu at (194.5, 69.8)
Connections:
- A1 pad A3: (no net) -> Net-(A1-PadA3)
- A1 pad A4: (no net) -> Net-(A1-PadA4)
- A1 pad A5: (no net) -> Net-(A1-PadA5)
- A1 pad D2: (no net) -> Net-(A1-PadD2)
- A1 pad D3: (no net) -> Net-(A1-PadD3)
- A1 pad D8: (no net) -> Net-(A1-PadD8)
- A1 pad EN: (no net) -> Net-(A1-PadEN)
- A1 pad LI+: (no net) -> Net-(A1-PadLI+)
- A1 pad MD: (no net) -> Net-(A1-PadMD)
- A1 pad MI: (no net) -> Net-(A1-PadMI)
- A1 pad MO: (no net) -> Net-(A1-PadMO)
- A1 pad RESET: (no net) -> Net-(A1-PadRESET)
- A1 pad RX: (no net) -> Net-(A1-PadRX)
- A1 pad SCK: (no net) -> Net-(A1-PadSCK)
- A1 pad TX: (no net) -> Net-(A1-PadTX)
- A1 pad VUSB: (no net) -> Net-(A1-PadVUSB)
- C3 pad 1: Enc-A -> Net-(C3-Pad1)
- C4 pad 2: Enc-B -> Net-(C4-Pad2)
- C5 pad 1: Enc-bt1 -> Net-(C5-Pad1)
- J2 pad 6: (no net) -> SWD-SWO
- J2 pad 7: (no net) -> Net-(J2-Pad7)
- J2 pad 8: (no net) -> Net-(J2-Pad8)
- J2 pad 9: (no net) -> Net-(J2-Pad9)
- SW2 pad A: Enc-A -> Net-(C3-Pad1)
- SW2 pad B: Enc-B -> Net-(C4-Pad2)
- SW2 pad S1: Enc-bt1 -> Net-(C5-Pad1)
- U6 pad 2: (no net) -> Net-(U6-Pad2)
- U6 pad 3: (no net) -> Net-(U6-Pad3)
- U6 pad 9: (no net) -> Net-(U6-Pad9)
