File: Horticulture.kicad_pcb (KiCad board)
At the start: 2 copper layers, 220 x 22 mm, 66 parts, among them J2 Conn_02x05_Odd_Even, J3 Conn_01x04_Male, J4 Conn_01x04_Male, SW1 SW-I2C, SW2 Rotary_Encoder_Switch, U1 TLE4309, U2 TLE4309, U3 TLE4309, U4 TLE4309, U6 STM32F030F4Px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

Commit message: Rev-3.2.1
Parts:
- R10, R7, R8, R9: footprint Resistor_SMD:R_0805_2012Metric_Pad1.15x1.40mm_HandSolder -> Resistor_SMD:R_0402_1005Metric
- R11: footprint Resistor_SMD:R_0603_1608Metric -> Resistor_SMD:R_0402_1005Metric
- R12, R13, R14, R15, R16, R17: footprint Resistor_SMD:R_0603_1608Metric -> Resistor_SMD:R_0402_1005Metric; moved to B.Cu
- moved R16 31.3 mm to (179.7, 89.8), turned to 180 degrees
- moved R17 27.6 mm to (185.5, 95.9)
- moved R15 26.0 mm to (179.7, 88.6), turned to 180 degrees
- moved R13 25.3 mm to (177.1, 83.1), turned to 180 degrees
- moved R14 20.7 mm to (179.7, 87.4), turned to 180 degrees
- moved R12 18.5 mm to (178.6, 81.5), turned to 180 degrees
- moved R11 5.55 mm to (64.3, 84.0), turned to 0 degrees
Connections:
- A1 pad A3: Net-(A1-PadA3) -> (no net)
- A1 pad A4: Net-(A1-PadA4) -> (no net)
- A1 pad A5: Net-(A1-PadA5) -> (no net)
- A1 pad D2: Net-(A1-PadD2) -> (no net)
- A1 pad D3: Net-(A1-PadD3) -> (no net)
- A1 pad D8: Net-(A1-PadD8) -> (no net)
- A1 pad EN: Net-(A1-PadEN) -> (no net)
- A1 pad LI+: Net-(A1-PadLI+) -> (no net)
- A1 pad MD: Net-(A1-PadMD) -> (no net)
- A1 pad MI: Net-(A1-PadMI) -> (no net)
- A1 pad MO: Net-(A1-PadMO) -> (no net)
- A1 pad RESET: Net-(A1-PadRESET) -> (no net)
- A1 pad RX: Net-(A1-PadRX) -> (no net)
- A1 pad SCK: Net-(A1-PadSCK) -> (no net)
- A1 pad TX: Net-(A1-PadTX) -> (no net)
- A1 pad VUSB: Net-(A1-PadVUSB) -> (no net)
- J2 pad 6: SWD-SWO -> (no net)
- J2 pad 7: Net-(J2-Pad7) -> (no net)
- J2 pad 8: Net-(J2-Pad8) -> (no net)
- J2 pad 9: Net-(J2-Pad9) -> (no net)
- U6 pad 2: Net-(U6-Pad2) -> (no net)
- U6 pad 3: Net-(U6-Pad3) -> (no net)
- U6 pad 9: Net-(U6-Pad9) -> (no net)
Routing:
- net Net-(C4-Pad2): track 0.00 -> 47.0 mm, vias 0 -> 2
- net Enc-B: track 168.3 -> 136.0 mm
- net Net-(C5-Pad1): track 0.00 -> 21.5 mm
- net +3.3V: track 216.0 -> 232.1 mm
- net Net-(C3-Pad1): track 0.00 -> 14.7 mm
- net Enc-A: track 143.6 -> 131.5 mm
- net SWD-GND: track 247.3 -> 257.3 mm, vias 17 -> 19
- net Enc-bt1: track 161.1 -> 152.9 mm, vias 1 -> 3
- net I2c-SDA: track 252.6 -> 256.8 mm, vias 3 -> 5
- net nRESET: track 12.4 -> 15.1 mm
- net I2c-SCL: track 240.0 -> 240.6 mm, vias 2 -> 4
- net UC-pwm4: track 184.2 -> 184.7 mm
- net UC-pwm3: track 171.7 -> 172.2 mm
- net UC-pwm1: track 95.9 -> 96.5 mm
Other:
- board text added: "Horticulture-rev-3.2.1"
- board text removed: "Horticulture-rev-3.1.2.0"
