File: Horticulture.kicad_pcb (KiCad board)
At the start: 2 copper layers, 220 x 22 mm, 66 parts, among them J2 Conn_02x05_Odd_Even, J3 Conn_01x04_Male, J4 Conn_01x04_Male, SW1 SW-I2C, SW2 Rotary_Encoder_Switch, U1 TLE4309, U2 TLE4309, U3 TLE4309, U4 TLE4309, U6 STM32F030F4Px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

Commit message: 3.2.1 RC1 Klar til Produksjon
Other:
- rule pad_to_mask_clearance: 0.05 -> 0

Commit message: 3.2.1- RC2. Fixes #4
Parts:
- added J1: Conn_01x04_Male, Connector_Molex:Molex_PicoBlade_53398-0471_1x04-1MP_P1.25mm_Vertical, B.Cu at (170.2, 91.2)
Routing:
- net I2c-SDA: track 256.8 -> 265.8 mm, vias 5 -> 7
- net I2c-SCL: track 240.6 -> 246.6 mm
- net +3.3V: track 232.1 -> 237.7 mm, vias 3 -> 4
- net SWD-GND: track 257.3 -> 262.7 mm
