File: Horticulture-LED/Horticulture.sch (KiCad schematic (older format))
At the start: 67 parts, among them J1 Conn_01x04_Male, J2 Conn_02x05_Odd_Even, J3 Conn_01x04_Male, J4 Conn_01x04_Male, SW1 SW-I2C, SW2 Rotary_Encoder_Switch, U1 TLE4309, U2 TLE4309, U3 TLE4309, U4 TLE4309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

Commit message: Fixed r-values for BOM
Parts:
- D1, D10, D11, D12, D13, D14, D15, D16, D17, D18, D19, D2, D20, D21, D22, D23, D24, D3, D4, D5, D6, D7, D8, D9: symbol test-rescue:LED-Device -> Horticulture-rescue:LED-Device-test-rescue
- R1, R2, R3, R4: value R_Small -> 0R39 current sense; symbol test-rescue:R_Small-Device -> Horticulture-rescue:R_Small-Device-test-rescue
- U1, U2, U3, U4: symbol test-rescue:TLE4309-Driver_LED -> Horticulture-rescue:TLE4309-Driver_LED-test-rescue
Changed lines of the file:
@@
 	2950 6100 2950 6300
 $Comp
-L test-rescue:GND-power #PWR0101
+L Horticulture-rescue:GND-power-test-rescue #PWR0101
 U 1 1 5EEF5ADC
 P 2950 6300
@@
 	8600 5850 8600 5950
 $Comp
-L test-rescue:R_Small-Device R4
+L Horticulture-rescue:R_Small-Device-test-rescue R4
 U 1 1 5EEED184
 P 8600 5750
 F 0 "R4" H 8659 5796 50  0000 L CNN
-F 1 "R_Small" H 8659 5705 50  0000 L CNN
+F 1 "0R39 current sense" H 8659 5705 50  0000 L CNN
 F 2 "Resistor_SMD:R_0805_2012Metric" H 8600 5750 50  0001 C CNN
 F 3 "~" H 8600 5750 50  0001 C CNN
@@
 $EndComp
 $Comp
-L test-rescue:TLE4309-Driver_LED U4
+L Horticulture-rescue:TLE4309-Driver_LED-test-rescue U4
 U 1 1 5EEDC8ED
 P 2950 5800
@@
 	8600 5550 8600 5650
 $Comp
-L test-rescue:GND-power #PWR0102
+L Horticulture-rescue:GND-power-test-rescue #PWR0102
 U 1 1 5EEC5AAB
 P 8600 5950
@@
 	2950 4600 2950 4800
 $Comp
-L test-rescue:GND-power #PWR0103
+L Horticulture-rescue:GND-power-test-rescue #PWR0103
 U 1 1 5EEFF231
 P 2950 4800
@@
 	8600 4350 8600 4450
 $Comp
-L test-rescue:R_Small-Device R3
+L Horticulture-rescue:R_Small-Device-test-rescue R3
 U 1 1 5EEFF240
 P 8600 4250
 F 0 "R3" H 8659 4296 50  0000 L CNN
-F 1 "R_Small" H 8659 4205 50  0000 L CNN
+F 1 "0R39 current sense" H 8659 4205 50  0000 L CNN
 F 2 "Resistor_SMD:R_0805_2012Metric" H 8600 4250 50  0001 C CNN
 F 3 "~" H 8600 4250 50  0001 C CNN
@@
 $EndComp
 $Comp
-L test-rescue:TLE4309-Driver_LED U3
+L Horticulture-rescue:TLE4309-Driver_LED-test-rescue U3
 U 1 1 5EEFF24B
 P 2950 4300
@@
 	8600 4050 8600 4150
 $Comp
-L test-rescue:GND-power #PWR0104
+L Horticulture-rescue:GND-power-test-rescue #PWR0104
 U 1 1 5EEFF258
 P 8600 4450
@@
 	2950 3200 2950 3400
 $Comp
-L test-rescue:GND-power #PWR0105
+L Horticulture-rescue:GND-power-test-rescue #PWR0105
 U 1 1 5EF0699A
 P 2950 3400
@@
 	8600 2950 8600 3050
 $Comp
-L test-rescue:R_Small-Device R2
+L Horticulture-rescue:R_Small-Device-test-rescue R2
 U 1 1 5EF069A9
 P 8600 2850
 F 0 "R2" H 8659 2896 50  0000 L CNN
-F 1 "R_Small" H 8659 2805 50  0000 L CNN
+F 1 "0R39 current sense" H 8659 2805 50  0000 L CNN
 F 2 "Resistor_SMD:R_0805_2012Metric" H 8600 2850 50  0001 C CNN
 F 3 "~" H 8600 2850 50  0001 C CNN
@@
 $EndComp
 $Comp
-L test-rescue:TLE4309-Driver_LED U2
+L Horticulture-rescue:TLE4309-Driver_LED-test-rescue U2
 U 1 1 5EF069B4
 P 2950 2900
@@
 	8600 2650 8600 2750
 $Comp
-L test-rescue:GND-power #PWR0106
+L Horticulture-rescue:GND-power-test-rescue #PWR0106
 U 1 1 5EF069C1
 P 8600 3050
@@
 	2950 1900 2950 2100
 $Comp
-L test-rescue:GND-power #PWR0107
+L Horticulture-rescue:GND-power-test-rescue #PWR0107
 U 1 1 5EF11D41
 P 2950 2100
@@
 	8600 1650 8600 1750
 $Comp
-L test-rescue:R_Small-Device R1
+L Horticulture-rescue:R_Small-Device-test-rescue R1
 U 1 1 5EF11D50
 P 8600 1550
 F 0 "R1" H 8659 1596 50  0000 L CNN
-F 1 "R_Small" H 8659 1505 50  0000 L CNN
+F 1 "0R39 current sense" H 8659 1505 50  0000 L CNN
 F 2 "Resistor_SMD:R_0805_2012Metric" H 8600 1550 50  0001 C CNN
 F 3 "~" H 8600 1550 50  0001 C CNN
@@
 	3350 1350 4400 1350
 $Comp
-L test-rescue:TLE4309-Driver_LED U1
+L Horticulture-rescue:TLE4309-Driver_LED-test-rescue U1
 U 1 1 5EF11D5B
 P 2950 1600
@@
 	8450 1350 8500 1350
 $Comp
-L test-rescue:GND-power #PWR0108
+L Horticulture-rescue:GND-power-test-rescue #PWR0108
 U 1 1 5EF11D68
 P 8600 1750
@@
 	4700 1350 5200 1350
 $Comp
-L test-rescue:LED-Device D6
+L Horticulture-rescue:LED-Device-test-rescue D6
 U 1 1 5EF11D77
 P 8300 1350
@@
 $EndComp
 $Comp
-L test-rescue:LED-Device D5
+L Horticulture-rescue:LED-Device-test-rescue D5
 U 1 1 5EF11D81
 P 7550 1350
@@
 $EndComp
 $Comp
-L test-rescue:LED-Device D4
+L Horticulture-rescue:LED-Device-test-rescue D4
 U 1 1 5EF11D8B
 P 6750 1350
@@
 $EndComp
 $Comp
-L test-rescue:LED-Device D3
+L Horticulture-rescue:LED-Device-test-rescue D3
 U 1 1 5EF11D95
 P 6000 1350
@@
 $EndComp
 $Comp
-L test-rescue:LED-Device D2
+L Horticulture-rescue:LED-Device-test-rescue D2
 U 1 1 5EF11D9F
 P 5350 1350
@@
 $EndComp
 $Comp
-L test-rescue:LED-Device D1
+L Horticulture-rescue:LED-Device-test-rescue D1
 U 1 1 5EF11DA9
 P 4550 1350
@@
 	4700 4050 5200 4050
 $Comp
-L test-rescue:LED-Device D18
+L Horticulture-rescue:LED-Device-test-rescue D18
 U 1 1 5EED18C4
 P 8300 4050
@@
 $EndComp
 $Comp
-L test-rescue:LED-Device D17
+L Horticulture-rescue:LED-Device-test-rescue D17
 U 1 1 5EED18CA
 P 7550 4050
@@
 $EndComp
 $Comp
-L test-rescue:LED-Device D16
+L Horticulture-rescue:LED-Device-test-rescue D16
 U 1 1 5EED18D0
 P 6750 4050
@@
 $EndComp
 $Comp
-L test-rescue:LED-Device D15
+L Horticulture-rescue:LED-Device-test-rescue D15
 U 1 1 5EED18D6
 P 6000 4050
@@
 $EndComp
 $Comp
-L test-rescue:LED-Device D14
+L Horticulture-rescue:LED-Device-test-rescue D14
 U 1 1 5EED18DC
 P 5350 4050
@@
 $EndComp
 $Comp
-L test-rescue:LED-Device D13
+L Horticulture-rescue:LED-Device-test-rescue D13
 U 1 1 5EED18E2
 P 4550 4050
@@
 	4700 5550 5200 5550
 $Comp
-L test-rescue:LED-Device D24
+L Horticulture-rescue:LED-Device-test-rescue D24
 U 1 1 5EED38D5
 P 8300 5550
@@
 $EndComp
 $Comp
-L test-rescue:LED-Device D23
+L Horticulture-rescue:LED-Device-test-rescue D23
 U 1 1 5EED38DB
 P 7550 5550
@@
 $EndComp
 $Comp
-L test-rescue:LED-Device D22
+L Horticulture-rescue:LED-Device-test-rescue D22
 U 1 1 5EED38E1
 P 6750 5550
@@
 $EndComp
 $Comp
-L test-rescue:LED-Device D21
+L Horticulture-rescue:LED-Device-test-rescue D21
 U 1 1 5EED38E7
 P 6000 5550
@@
 $EndComp
 $Comp
-L test-rescue:LED-Device D20
+L Horticulture-rescue:LED-Device-test-rescue D20
 U 1 1 5EED38ED
 P 5350 5550
@@
 $EndComp
 $Comp
-L test-rescue:LED-Device D19
+L Horticulture-rescue:LED-Device-test-rescue D19
 U 1 1 5EED38F3
 P 4550 5550
@@
 $EndComp
 $Comp
-L test-rescue:LED-Device D7
+L Horticulture-rescue:LED-Device-test-rescue D7
 U 1 1 5EECB202
 P 4550 2650
@@
 $EndComp
 $Comp
-L test-rescue:LED-Device D8
+L Horticulture-rescue:LED-Device-test-rescue D8
 U 1 1 5EECB1F8
 P 5350 2650
@@
 $EndComp
 $Comp
-L test-rescue:LED-Device D9
+L Horticulture-rescue:LED-Device-test-rescue D9
 U 1 1 5EECB1EE
 P 6000 2650
@@
 $EndComp
 $Comp
-L test-rescue:LED-Device D10
+L Horticulture-rescue:LED-Device-test-rescue D10
 U 1 1 5EECB1E4
 P 6750 2650
@@
 $EndComp
 $Comp
-L test-rescue:LED-Device D11
+L Horticulture-rescue:LED-Device-test-rescue D11
 U 1 1 5EECB1DA
 P 7550 2650
@@
 $EndComp
 $Comp
-L test-rescue:LED-Device D12
+L Horticulture-rescue:LED-Device-test-rescue D12
 U 1 1 5EECB1D0
 P 8300 2650
@@
 Connection ~ 8500 5550
 $Comp
-L test-rescue:VDC-power #PWR0109
+L Horticulture-rescue:VDC-power-test-rescue #PWR0109
 U 1 1 5EF8E4D7
 P 2550 1500
@@
 $EndComp
 $Comp
-L test-rescue:VDC-power #PWR0110
+L Horticulture-rescue:VDC-power-test-rescue #PWR0110
 U 1 1 5EF8EE2A
 P 2550 2800
@@
 $EndComp
 $Comp
-L test-rescue:VDC-power #PWR0111
+L Horticulture-rescue:VDC-power-test-rescue #PWR0111
 U 1 1 5EF8F8CE
 P 2550 4200
@@
 $EndComp
 $Comp
-L test-rescue:VDC-power #PWR0112
+L Horticulture-rescue:VDC-power-test-rescue #PWR0112
 U 1 1 5EF9014F
 P 2550 5700
@@
 	12950 7700 12950 7800
 $Comp
-L test-rescue:GND-power #PWR0113
+L Horticulture-rescue:GND-power-test-rescue #PWR0113
 U 1 1 5F5E9A88
 P 11600 4500

Commit message: Fixed resistor values
Parts:
- D6: value LED -> LED-purple
- R1: value 0R39 current sense -> 1ohm
- Renb1: value 200k -> 10k
- Rent1: value 412k -> 10k
Changed lines of the file:
@@
 P 8600 1550
 F 0 "R1" H 8659 1596 50  0000 L CNN
-F 1 "0R39 current sense" H 8659 1505 50  0000 L CNN
+F 1 "1ohm" H 8659 1505 50  0000 L CNN
 F 2 "Resistor_SMD:R_0805_2012Metric" H 8600 1550 50  0001 C CNN
 F 3 "~" H 8600 1550 50  0001 C CNN
@@
 P 8300 1350
 F 0 "D6" H 8293 1567 50  0000 C CNN
-F 1 "LED" H 8293 1476 50  0000 C CNN
+F 1 "LED-purple" H 8293 1476 50  0000 C CNN
 F 2 "LED_SMD:Sunplus-35" H 8300 1350 50  0001 C CNN
 F 3 "~" H 8300 1350 50  0001 C CNN
@@
 P 3300 8150
 F 0 "Renb1" H 3370 8196 50  0000 L CNN
-F 1 "200k" H 3370 8105 50  0000 L CNN
+F 1 "10k" H 3370 8105 50  0000 L CNN
 F 2 "Resistor_SMD:R_0402_1005Metric" V 3230 8150 50  0001 C CNN
 F 3 "~" H 3300 8150 50  0001 C CNN
@@
 P 3300 7400
 F 0 "Rent1" H 3370 7446 50  0000 L CNN
-F 1 "412k" H 3370 7355 50  0000 L CNN
+F 1 "10k" H 3370 7355 50  0000 L CNN
 F 2 "Resistor_SMD:R_0402_1005Metric" V 3230 7400 50  0001 C CNN
 F 3 "~" H 3300 7400 50  0001 C CNN

Commit message: Picoblade connector added for stm programming, minor bug fixes
Parts:
- removed J2: Conn_02x05_Odd_Even, Connector_PinHeader_1.27mm:PinHeader_2x05_P1.27mm_Vertical_SMD, symbol Connector_Generic:Conn_02x05_Odd_Even
- added Prgrm1: Conn_01x04_Male, Connector_Molex:Molex_PicoBlade_53398-0471_1x04-1MP_P1.25mm_Vertical, symbol Connector:Conn_01x04_Male
- R2, R3, R4: value 0R39 current sense -> 1ohm
Connections:
- net labels removed: SWD-GND, SWD-SWO, SWD-VDD-Target
- wire segments 138 -> 132
Changed lines of the file:
@@
 	8600 5850 8600 5950
-$Comp
-L Horticulture-rescue:R_Small-Device-test-rescue R4
-U 1 1 5EEED184
-P 8600 5750
-F 0 "R4" H 8659 5796 50  0000 L CNN
-F 1 "0R39 current sense" H 8659 5705 50  0000 L CNN
-F 2 "Resistor_SMD:R_0805_2012Metric" H 8600 5750 50  0001 C CNN
-F 3 "~" H 8600 5750 50  0001 C CNN
-	1    8600 5750
-	1    0    0    -1
-$EndComp
 $Comp
 L Horticulture-rescue:TLE4309-Driver_LED-test-rescue U4
@@
 P 8600 4250
 F 0 "R3" H 8659 4296 50  0000 L CNN
-F 1 "0R39 current sense" H 8659 4205 50  0000 L CNN
+F 1 "1ohm" H 8659 4205 50  0000 L CNN
 F 2 "Resistor_SMD:R_0805_2012Metric" H 8600 4250 50  0001 C CNN
 F 3 "~" H 8600 4250 50  0001 C CNN
@@
 P 8600 2850
 F 0 "R2" H 8659 2896 50  0000 L CNN
-F 1 "0R39 current sense" H 8659 2805 50  0000 L CNN
+F 1 "1ohm" H 8659 2805 50  0000 L CNN
 F 2 "Resistor_SMD:R_0805_2012Metric" H 8600 2850 50  0001 C CNN
 F 3 "~" H 8600 2850 50  0001 C CNN
@@
 	1    0    0    -1
 $EndComp
-$Comp
-L Connector_Generic:Conn_02x05_Odd_Even J2
-U 1 1 5EF0F96A
-P 13150 8000
-F 0 "J2" H 13200 8417 50  0000 C CNN
-F 1 "Conn_02x05_Odd_Even" H 13200 8326 50  0000 C CNN
-F 2 "Connector_PinHeader_1.27mm:PinHeader_2x05_P1.27mm_Vertical_SMD" H 13150 8000 50  0001 C CNN
-F 3 "~" H 13150 8000 50  0001 C CNN
-	1    13150 8000
-	1    0    0    -1
-$EndComp
-Text GLabel 12950 7800 0    50   Input ~ 0
-SWD-VDD-Target
-Text GLabel 13450 8200 2    50   Input ~ 0
-nRESET
-Text GLabel 13450 8000 2    50   Input ~ 0
-SWD-SWO
-Text GLabel 13450 7900 2    50   Input ~ 0
+Text GLabel 13150 7750 0    50   Input ~ 0
 SWD-SWCLK
-Text GLabel 13450 7800 2    50   Input ~ 0
+Text GLabel 13150 7650 0    50   Input ~ 0
 SWD-SWIO
-Text GLabel 12950 7900 0    50   Input ~ 0
-SWD-GND
-Wire Wire Line
-	12950 8000 12950 7900
-$Comp
-L power:GND #PWR0118
-U 1 1 5EF17CE3
-P 12600 8050
-F 0 "#PWR0118" H 12600 7800 50  0001 C CNN
-F 1 "GND" H 12605 7877 50  0000 C CNN
-F 2 "" H 12600 8050 50  0001 C CNN
-F 3 "" H 12600 8050 50  0001 C CNN
-	1    12600 8050
-	1    0    0    -1
-$EndComp
-Wire Wire Line
-	12600 8050 12750 8050
-Wire Wire Line
-	12750 8050 12750 8000
-Wire Wire Line
-	12750 8000 12950 8000
-Connection ~ 12950 8000
 Text GLabel 7450 7150 0    50   Input ~ 0
 nRESET
@@
 Text GLabel 1100 1550 2    50   Input ~ 0
 VDC
-Text GLabel 1100 1650 2    50   Input ~ 0
-SWD-GND
 Text GLabel 11600 1850 1    50   Input ~ 0
 +3.3V
@@
 Text GLabel 1100 2150 2    50   Input ~ 0
 VDC
-Text GLabel 1100 2250 2    50   Input ~ 0
-SWD-GND
-Text GLabel 12750 7700 0    50   Input ~ 0
+Text GLabel 13150 7550 0    50   Input ~ 0
 +3.3V
-Wire Wire Line
-	12750 7700 12950 7700
-Wire Wire Line
-	12950 7700 12950 7800
 $Comp
 L Horticulture-rescue:GND-power-test-rescue #PWR0113
@@
 	-1   0    0    1
 $EndComp
+$Comp
+L power:GND #PWR0118
+U 1 1 600C4853
+P 13150 7850
+F 0 "#PWR0118" H 13150 7600 50  0001 C CNN
+F 1 "GND" H 13155 7677 50  0000 C CNN
+F 2 "" H 13150 7850 50  0001 C CNN
+F 3 "" H 13150 7850 50  0001 C CNN
+	1    13150 7850
+	0    1    1    0
+$EndComp
+$Comp
+L power:GND #PWR0127
+U 1 1 600D22E3
+P 1100 2250
+F 0 "#PWR0127" H 1100 2000 50  0001 C CNN
+F 1 "GND" H 1105 2077 50  0000 C CNN
+F 2 "" H 1100 2250 50  0001 C CNN
+F 3 "" H 1100 2250 50  0001 C CNN
+	1    1100 2250
+	0    -1   -1   0
+$EndComp
+$Comp
+L power:GND #PWR0128
+U 1 1 600D36DB
+P 1100 1650
+F 0 "#PWR0128" H 1100 1400 50  0001 C CNN
+F 1 "GND" H 1105 1477 50  0000 C CNN
+F 2 "" H 1100 1650 50  0001 C CNN
+F 3 "" H 1100 1650 50  0001 C CNN
+	1    1100 1650
+	0    -1   -1   0
+$EndComp
+$Comp
+L Connector:Conn_01x04_Male Prgrm1
+U 1 1 6008A5A0
+P 13350 7750
+F 0 "Prgrm1" H 13322 7632 50  0000 R CNN
+F 1 "Conn_01x04_Male" H 13322 7723 50  0000 R CNN
+F 2 "Connector_Molex:Molex_PicoBlade_53398-0471_1x04-1MP_P1.25mm_Vertical" H 13350 7750 50  0001 C CNN
+F 3 "~" H 13350 7750 50  0001 C CNN
+	1    13350 7750
+	-1   0    0    1
+$EndComp
+$Comp
+L Horticulture-rescue:R_Small-Device-test-rescue R4
+U 1 1 5EEED184
+P 8600 5750
+F 0 "R4" H 8659 5796 50  0000 L CNN
+F 1 "1ohm" H 8659 5705 50  0000 L CNN
+F 2 "Resistor_SMD:R_0805_2012Metric" H 8600 5750 50  0001 C CNN
+F 3 "~" H 8600 5750 50  0001 C CNN
+	1    8600 5750
+	1    0    0    -1
+$EndComp
 $EndSCHEMATC

Commit message: Added CI/CD, changed rev in notes to rev in silk layer
And cleaned repo
Connections:
- net labels added: nReset
- net labels removed: nRESET
- wire segments 132 -> 133
- no-connect marks 0 -> 27
Changed lines of the file:
@@
 Sheet 1 1
 Title "Horticulture LED"
-Date "2020-12-06"
-Rev "3.2.1"
+Date "2021-06-15"
+Rev "3.3.1"
 Comp "Horticulture project"
 Comment1 ""
@@
 Text GLabel 13150 7650 0    50   Input ~ 0
 SWD-SWIO
-Text GLabel 7450 7150 0    50   Input ~ 0
-nRESET
 Text GLabel 8650 8250 2    50   Input ~ 0
 SWD-SWCLK
@@
 $EndComp
 Wire Wire Line
-	7450 7150 7600 7150
-Wire Wire Line
 	7600 7050 7600 7150
-Connection ~ 7600 7150
 Wire Wire Line
 	7600 7150 7650 7150
-Wire Wire Line
-	7600 6850 8200 6850
 Wire Wire Line
 	8200 6850 8200 6950
@@
 	1    0    0    -1
 $EndComp
+$Comp
+L power:PWR_FLAG #FLG0101
+U 1 1 60C84C4E
+P 2280 1500
+F 0 "#FLG0101" H 2280 1575 50  0001 C CNN
+F 1 "PWR_FLAG" H 2280 1673 50  0000 C CNN
+F 2 "" H 2280 1500 50  0001 C CNN
+F 3 "~" H 2280 1500 50  0001 C CNN
+	1    2280 1500
+	1    0    0    -1
+$EndComp
+Wire Wire Line
+	2550 1500 2280 1500
+Connection ~ 2550 1500
+NoConn ~ 7650 7950
+NoConn ~ 7650 8050
+NoConn ~ 8650 7450
+NoConn ~ 12600 1800
+NoConn ~ 14050 1950
+NoConn ~ 14050 2100
+NoConn ~ 13300 2450
+NoConn ~ 13300 2600
+NoConn ~ 13300 2750
+NoConn ~ 13300 2900
+NoConn ~ 12600 1900
+NoConn ~ 12400 1500
+NoConn ~ 12300 1500
+NoConn ~ 12200 1500
+NoConn ~ 12000 1500
+NoConn ~ 10350 4100
+NoConn ~ 10350 3950
+NoConn ~ 10350 3800
+NoConn ~ 10350 3650
+NoConn ~ 10350 3500
+NoConn ~ 10350 3050
+NoConn ~ 10350 3200
+NoConn ~ 10350 3350
+NoConn ~ 10350 2300
+NoConn ~ 10350 2450
+$Comp
+L power:PWR_FLAG #FLG0102
+U 1 1 60D5B8D8
+P 7760 6850
+F 0 "#FLG0102" H 7760 6925 50  0001 C CNN
+F 1 "PWR_FLAG" H 7760 7023 50  0000 C CNN
+F 2 "" H 7760 6850 50  0001 C CNN
+F 3 "~" H 7760 6850 50  0001 C CNN
+	1    7760 6850
+	1    0    0    -1
+$EndComp
+Connection ~ 7760 6850
+Wire Wire Line
+	7760 6850 8200 6850
+Wire Wire Line
+	7600 6850 7760 6850
+NoConn ~ 13300 3650
+NoConn ~ 13300 3800
+Text Label 7335 7180 0    50   ~ 0
+nReset
 $EndSCHEMATC

Commit message: More i2c connectors added, fp for 12c/pwm added, removed stm 32 fp, moved tle drivers
Parts:
- removed C3, C4, C5: 100nF, Capacitor_SMD:C_0603_1608Metric, symbol Device:C_Small
- removed J1: Conn_01x04_Male, Connector_Molex:Molex_PicoBlade_53398-0471_1x04-1MP_P1.25mm_Vertical, symbol Connector:Conn_01x04_Male
- removed R11, R12, R13, R14, R15, R16, R17: 10K2, Resistor_SMD:R_0402_1005Metric, symbol Device:R_Small
- removed SW1: SW-I2C, Jumper:SolderJumper-2_P1.3mm_Open_RoundedPad1.0x1.5mm, symbol Switch:SW_DIP_x01
- removed SW2: Rotary_Encoder_Switch, Rotary_Encoder:EC11J1524413-modiied, symbol Device:Rotary_Encoder_Switch
- removed U6: STM32F030F4Px, Package_SO:TSSOP-20_4.4x6.5mm_P0.65mm, symbol MCU_ST_STM32F0:STM32F030F4Px
- removed U7: SSD1306, Connector_PinHeader_2.54mm:PinHeader_1x04_P2.54mm_Vertical, symbol SSD1306_OLED-0.91-128x32:SSD1306
- added 3.3v_i2c2, 3.3v_i2c3, 3.3v_i2c4: Conn_01x04_Male, Connector_Molex:Molex_PicoBlade_53398-0471_1x04-1MP_P1.25mm_Vertical, symbol Connector:Conn_01x04_Male
- added D25, D26, D27, D28, D29, D30, D31, D32: LED, LED_SMD:Sunplus-2835, symbol Horticulture-rescue:LED-Device-test-rescue
- added JP1: i2c addr 1, Jumper:SolderJumper-3_P1.3mm_Bridged12_RoundedPad1.0x1.5mm_NumberLabels, symbol Jumper:SolderJumper_3_Bridged12
- added JP2: i2c addr 2, Jumper:SolderJumper-3_P1.3mm_Bridged12_RoundedPad1.0x1.5mm_NumberLabels, symbol Jumper:SolderJumper_3_Bridged12
- added U5: PCA9633DP2, Package_TO_SOT_SMD:SOT-552-1-nxp, symbol Horticulture-rescue:nrf-led-feather-rescue_PCA9633DP2-i2c-led-feather-cache
- D1, D10, D11, D12, D13, D14, D15, D16, D17, D18, D19, D2, D20, D21, D22, D23, D24, D3, D4, D5, D7, D8, D9: footprint LED_SMD:Sunplus-35 -> LED_SMD:Sunplus-2835
- D6: value LED-purple -> LED; footprint LED_SMD:Sunplus-35 -> LED_SMD:Sunplus-2835
- U1, U2, U3, U4: Supplier (none) -> https://no.rs-online.com/web/p/led-driver-ics/0492957/
- VR1: Supplier (none) -> https://www.digikey.no/product-detail/no/texas-instruments/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
- renumbered Prgrm1 to 3.3v_i2c1, D25 to D33
Connections:
- net labels added: +24vdc
- net labels removed: Enc-A, Enc-B, Enc-bt1, SWD-SWCLK, SWD-SWIO, VDC, i2c-addr, nReset
- wire segments 133 -> 108
Other:
- note added: "3.3v generator"
- note added: "Led driver array"
- note added: "Main board connector"
- note added: "i2c outputs (picoblade)"
- note added: "i2c-PWM module"
- moved on the sheet: 3.3v_i2c1, Cboot1, Cin1, Cinx1, Cout1, D1, D10, D11, D12, D13, D14, D15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
