File: Horticulture-LED/Horticulture.kicad_pcb (KiCad board)
At the start: 2 copper layers, 220 x 22 mm, 61 parts, among them J3 Conn_01x04_Male, J4 Conn_01x04_Male, U1 TLE4309, U2 TLE4309, U3 TLE4309, U4 TLE4309, U5 PCA9633DP2, U6 MCP1703A-1502_SOT223

Commit message: esd-modboard
Parts:
- moved R4 2.08 mm to (256.8, 96.5)
- moved R1 1.74 mm to (256.8, 85.3)
Routing:
- net Net-(D8-Pad1): track 157.0 -> 147.6 mm
Other:
- rule pad_to_mask_clearance: 0 -> -0.3

Commit message: Updated to KiCad6
Other:
- net class Default removed
- net class Led-Driver removed
- net class Led-power removed
- net class VDC removed
- net class ymse power removed
