File: Horticulture-LED/Horticulture-LED.kicad_pcb (KiCad board)
At the start: 2 copper layers, 220 x 22 mm, 61 parts, among them J3 Conn_01x04_Male, J4 Conn_01x04_Male, U1 TLE4309, U2 TLE4309, U3 TLE4309, U4 TLE4309, U5 PCA9633DP2, U6 MCP1703A-1502_SOT223

Commit message: Updated component reference
Parts:
- renumbered 3.3v_i2c1 to 3_3v_i2c1, 3.3v_i2c2 to 3_3v_i2c2, 3.3v_i2c4 to 3_3v_i2c3, 3.3v_i2c3 to 3_3v_i2c4
Changed lines of the file:
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@@
 		(descr "Molex PicoBlade series connector, 53398-0471 (http://www.molex.com/pdm_docs/sd/533980271_sd.pdf), generated with kicad-footprint-generator")
 		(tags "connector Molex PicoBlade side entry")
-		(property "Reference" "3.3v_i2c4"
+		(property "Reference" "3_3v_i2c3"
 			(at 0 3.1 90)
 			(layer "B.SilkS")
@@
 		)
 		(property "Footprint" ""
-			(at 0 0 -90)
+			(at 0 0 90)
 			(layer "F.Fab")
 			(hide yes)
@@
 		)
 		(property "Datasheet" ""
-			(at 0 0 -90)
+			(at 0 0 90)
 			(layer "F.Fab")
 			(hide yes)
@@
 		)
 		(property "Description" ""
-			(at 0 0 -90)
+			(at 0 0 90)
 			(layer "F.Fab")
 			(hide yes)
@@
 		(descr "Molex PicoBlade series connector, 53398-0471 (http://www.molex.com/pdm_docs/sd/533980271_sd.pdf), generated with kicad-footprint-generator")
 		(tags "connector Molex PicoBlade side entry")
-		(property "Reference" "3.3v_i2c2"
+		(property "Reference" "3_3v_i2c2"
 			(at 0 3.1 90)
 			(layer "B.SilkS")
@@
 		)
 		(property "Footprint" ""
-			(at 0 0 -90)
+			(at 0 0 90)
 			(layer "F.Fab")
 			(hide yes)
@@
 		)
 		(property "Datasheet" ""
-			(at 0 0 -90)
+			(at 0 0 90)
 			(layer "F.Fab")
 			(hide yes)
@@
 		)
 		(property "Description" ""
-			(at 0 0 -90)
+			(at 0 0 90)
 			(layer "F.Fab")
 			(hide yes)
@@
 		(descr "Molex PicoBlade series connector, 53398-0471 (http://www.molex.com/pdm_docs/sd/533980271_sd.pdf), generated with kicad-footprint-generator")
 		(tags "connector Molex PicoBlade side entry")
-		(property "Reference" "3.3v_i2c3"
+		(property "Reference" "3_3v_i2c4"
 			(at 0 3.1 90)
 			(layer "B.SilkS")
@@
 		)
 		(property "Footprint" ""
-			(at 0 0 -90)
+			(at 0 0 90)
 			(layer "F.Fab")
 			(hide yes)
@@
 		)
 		(property "Datasheet" ""
-			(at 0 0 -90)
+			(at 0 0 90)
 			(layer "F.Fab")
 			(hide yes)
@@
 		)
 		(property "Description" ""
-			(at 0 0 -90)
+			(at 0 0 90)
 			(layer "F.Fab")
 			(hide yes)
@@
 		(descr "Molex PicoBlade series connector, 53398-0471 (http://www.molex.com/pdm_docs/sd/533980271_sd.pdf), generated with kicad-footprint-generator")
 		(tags "connector Molex PicoBlade side entry")
-		(property "Reference" "3.3v_i2c1"
+		(property "Reference" "3_3v_i2c1"
 			(at 0 3.1 90)
 			(layer "B.SilkS")
@@
 		)
 		(property "Footprint" ""
-			(at 0 0 -90)
+			(at 0 0 90)
 			(layer "F.Fab")
 			(hide yes)
@@
 		)
 		(property "Datasheet" ""
-			(at 0 0 -90)
+			(at 0 0 90)
 			(layer "F.Fab")
 			(hide yes)
@@
 		)
 		(property "Description" ""
-			(at 0 0 -90)
+			(at 0 0 90)
 			(layer "F.Fab")
 			(hide yes)

Commit message: Fixed 3.3V i2c references
Parts:
- renumbered 3_3v_i2c1 to J1, 3_3v_i2c2 to J2, 3_3v_i2c3 to J5, 3_3v_i2c4 to J6
Changed lines of the file:
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@@
 		(descr "Molex PicoBlade series connector, 53398-0471 (http://www.molex.com/pdm_docs/sd/533980271_sd.pdf), generated with kicad-footprint-generator")
 		(tags "connector Molex PicoBlade side entry")
-		(property "Reference" "3_3v_i2c3"
+		(property "Reference" "J5"
 			(at 0 3.1 90)
 			(layer "B.SilkS")
@@
 		(descr "Molex PicoBlade series connector, 53398-0471 (http://www.molex.com/pdm_docs/sd/533980271_sd.pdf), generated with kicad-footprint-generator")
 		(tags "connector Molex PicoBlade side entry")
-		(property "Reference" "3_3v_i2c2"
+		(property "Reference" "J2"
 			(at 0 3.1 90)
 			(layer "B.SilkS")
@@
 		(descr "Molex PicoBlade series connector, 53398-0471 (http://www.molex.com/pdm_docs/sd/533980271_sd.pdf), generated with kicad-footprint-generator")
 		(tags "connector Molex PicoBlade side entry")
-		(property "Reference" "3_3v_i2c4"
+		(property "Reference" "J6"
 			(at 0 3.1 90)
 			(layer "B.SilkS")
@@
 		(descr "Molex PicoBlade series connector, 53398-0471 (http://www.molex.com/pdm_docs/sd/533980271_sd.pdf), generated with kicad-footprint-generator")
 		(tags "connector Molex PicoBlade side entry")
-		(property "Reference" "3_3v_i2c1"
+		(property "Reference" "J1"
 			(at 0 3.1 90)
 			(layer "B.SilkS")
