File: esd-modboard/esd-modboard/esd-modboard.kicad_pcb (KiCad board)
At the start: 2 copper layers, 5.3 x 8.6 mm, 2 parts, among them J1 Conn_01x04_Female

Commit message: Updated to kicad 8
Other:
- net class Default removed
